File: jogs.kicad_sch (KiCad schematic)
At the start: 3 parts, among them SW1 RotaryEncoder, SW3 RotaryEncoder_Switch, SW4 RotaryEncoder

Commit message: Add files via upload
Parts:
- removed SW3: RotaryEncoder_Switch, symbol Device:RotaryEncoder_Switch
- removed SW4: RotaryEncoder, symbol Device:RotaryEncoder
- added C1, C2, C3, C4, C5, C6: 10nF, Capacitor_SMD:C_0603_1608Metric, symbol Device:C_Small
- added J2: Conn_01x03_Pin, Connector_PinHeader_2.54mm:PinHeader_1x03_P2.54mm_Horizontal, symbol Connector:Conn_01x03_Pin
- added R10, R11, R12, R13, R14, R3, R4, R5, R6, R7, R8, R9: 10k, Resistor_SMD:R_0603_1608Metric, symbol Device:R_Small_US
- added SW2: RotaryEncoder_Switch, PEC11R_4215F_S0024:XDCR_PEC11R-4215F-S0024, symbol Device:RotaryEncoder_Switch
- added SW3: RotaryEncoder, footprints:PEC11R-4x15F-Nxxxx_BRN, symbol Device:RotaryEncoder
- SW1: footprint (none) -> footprints:PEC11R-4x15F-Nxxxx_BRN
Connections:
- net GND: now also SW1.2 (C), C1.2, C2.1, C3.1, C4.2, C5.1, C6.2, SW2.1 (S1), SW2.COM (C), SW3.2 (C); no longer SW1.C
- net JOG_1_A_LINE: now also C1.1, R3.1; no longer SW1.A
- net JOG_1_B_LINE: now also C2.2, R4.2; no longer SW1.B
- net JOG_2_A_LINE: now also C6.1, R14.1
- net JOG_2_B_LINE: now also C5.2, R13.2
- net SONG_SELECTOR_A_LINE: now also C3.2, R7.2
- net SONG_SELECTOR_B_LINE: now also C4.1, R10.1
- net SONG_SELECTOR_SWITCH: now also SW2.2 (S2)
- new net: R12.2, R14.2, SW3.1 (A)
- new net: R11.1, R13.1, SW3.3 (B)
- new net: R3.2, R5.2, SW1.1 (A)
- new net: R4.1, R6.1, SW1.3 (B)
- new net: R7.1, R8.1, SW2.A
- new net: R10.2, R9.2, SW2.B
- new net +3V3: R11.2, R12.1, R5.1, R6.2, R8.2, R9.1
- new net CAPACITIVE_SENSE_JOG_1: J2.2 (Pin_2)
- new net CAPACITIVE_SENSE_JOG_2: J2.3 (Pin_3)
- new net SEND_PIN_CAPACITIVE: J2.1 (Pin_1)
Other:
- note removed: "NEED TO ADD RC FILTER CIRCUIT ONCE ROTARY ENCODER IS DECIDED"
- company: Alex Goldberg -> Alex G
- title: MiniMixer -> @opensourcedj on twitter
- moved on the sheet: SW1
