File: leds.kicad_sch (KiCad schematic)
At the start: 33 parts

Commit message: Add files via upload
Parts:
- added C12, C15, C18, C21, C24, C27, C30, C31, C32, C33, C34, C35, C9: 100nF, Capacitor_SMD:C_0603_1608Metric, symbol Device:C_Small
- added D12, D15, D18, D21, D24, D25, D26, D27, D28, D3, D6, D9: WS2812B_passive_vss, LED_SMD:LED_WS2812B_PLCC4_5.0x5.0mm_P3.2mm, symbol LED:WS2812B_passive_vss
- added U2: CD74HCT125M96, footprints_CD74HCT125M96:D14, symbol 2025-06-01_06-17-26:CD74HCT125M96
- C10: renamed from C2; footprint (none) -> Capacitor_SMD:C_0603_1608Metric
- C11: renamed from C10; footprint (none) -> Capacitor_SMD:C_0603_1608Metric
- C13: renamed from C3; footprint (none) -> Capacitor_SMD:C_0603_1608Metric
- C14: renamed from C11; footprint (none) -> Capacitor_SMD:C_0603_1608Metric
- C16: renamed from C4; footprint (none) -> Capacitor_SMD:C_0603_1608Metric
- C17: renamed from C12; footprint (none) -> Capacitor_SMD:C_0603_1608Metric
- C19: renamed from C5; footprint (none) -> Capacitor_SMD:C_0603_1608Metric
- C20: renamed from C13; footprint (none) -> Capacitor_SMD:C_0603_1608Metric
- C22: renamed from C7; footprint (none) -> Capacitor_SMD:C_0603_1608Metric
- C23: renamed from C14; footprint (none) -> Capacitor_SMD:C_0603_1608Metric
- C25: renamed from C8; footprint (none) -> Capacitor_SMD:C_0603_1608Metric
- C26: renamed from C15; footprint (none) -> Capacitor_SMD:C_0603_1608Metric
- C28: renamed from C9; footprint (none) -> Capacitor_SMD:C_0603_1608Metric
- C29: renamed from C16; footprint (none) -> Capacitor_SMD:C_0603_1608Metric
- C7: renamed from C1; footprint (none) -> Capacitor_SMD:C_0603_1608Metric
- C8: renamed from C6; footprint (none) -> Capacitor_SMD:C_0603_1608Metric
- D1: value WS2812B -> WS2812B_passive_vss; symbol LED:WS2812B -> LED:WS2812B_passive_vss
- D10: renamed from D4; value WS2812B -> WS2812B_passive_vss; symbol LED:WS2812B -> LED:WS2812B_passive_vss
- D11: renamed from D12; value WS2812B -> WS2812B_passive_vss; symbol LED:WS2812B -> LED:WS2812B_passive_vss
- D13: renamed from D5; value WS2812B -> WS2812B_passive_vss; symbol LED:WS2812B -> LED:WS2812B_passive_vss
- D14: renamed from D13; value WS2812B -> WS2812B_passive_vss; symbol LED:WS2812B -> LED:WS2812B_passive_vss
- D16: renamed from D6; value WS2812B -> WS2812B_passive_vss; symbol LED:WS2812B -> LED:WS2812B_passive_vss
- D17: renamed from D14; value WS2812B -> WS2812B_passive_vss; symbol LED:WS2812B -> LED:WS2812B_passive_vss
- D19: renamed from D7; value WS2812B -> WS2812B_passive_vss; symbol LED:WS2812B -> LED:WS2812B_passive_vss
- D2: renamed from D9; value WS2812B -> WS2812B_passive_vss; symbol LED:WS2812B -> LED:WS2812B_passive_vss
- D20: renamed from D15; value WS2812B -> WS2812B_passive_vss; symbol LED:WS2812B -> LED:WS2812B_passive_vss
- D22: renamed from D8; value WS2812B -> WS2812B_passive_vss; symbol LED:WS2812B -> LED:WS2812B_passive_vss
- D23: renamed from D16; value WS2812B -> WS2812B_passive_vss; symbol LED:WS2812B -> LED:WS2812B_passive_vss
- D4: renamed from D2; value WS2812B -> WS2812B_passive_vss; symbol LED:WS2812B -> LED:WS2812B_passive_vss
- D5: renamed from D10; value WS2812B -> WS2812B_passive_vss; symbol LED:WS2812B -> LED:WS2812B_passive_vss
- D7: renamed from D3; value WS2812B -> WS2812B_passive_vss; symbol LED:WS2812B -> LED:WS2812B_passive_vss
- D8: renamed from D11; value WS2812B -> WS2812B_passive_vss; symbol LED:WS2812B -> LED:WS2812B_passive_vss
- R15: renamed from R1; value 330 -> 330 ohm; footprint (none) -> Resistor_SMD:R_0603_1608Metric
Connections:
- net GND: now also C12.2, C15.2, C18.2, C21.2, C24.2, C27.2, C30.2, C31.2, C32.2, C33.2, C34.2, C35.2, C9.2, D12.3 (VSS), D15.3 (VSS), D18.3 (VSS), D21.3 (VSS), D24.3 (VSS), D25.3 (VSS), D26.3 (VSS), D27.3 (VSS), D28.3 (VSS), D3.3 (VSS), D6.3 (VSS), D9.3 (VSS), U2.1 (*1OE), U2.7 (GND)
- net at D5.2 (DOUT), D8.4 (DIN): no longer C11.1
- net at D4.2 (DOUT), D7.4 (DIN): no longer C10.1
- net at D23.4 (DIN): now also D20.2 (DOUT)
- net at D22.4 (DIN): now also D19.2 (DOUT)
- net at R15.1: now also U2.3 (1Y)
- net 5V renamed 5V_POWER_BANK
- net 5V_POWER_BANK: now also C10.1, C11.1, C12.1, C15.1, C18.1, C21.1, C24.1, C27.1, C30.1, C31.1, C32.1, C33.1, C34.1, C35.1, C9.1, D12.1 (VDD), D15.1 (VDD), D18.1 (VDD), D21.1 (VDD), D24.1 (VDD), D25.1 (VDD), D26.1 (VDD), D27.1 (VDD), D28.1 (VDD), D3.1 (VDD), D6.1 (VDD), D9.1 (VDD), U2.10 (*3OE), U2.13 (*4OE), U2.14 (VCC), U2.4 (*2OE); no longer D10.2 (DOUT), D10.4 (DIN), D11.2 (DOUT), D11.4 (DIN), D13.2 (DOUT), D13.4 (DIN), D14.2 (DOUT), D14.4 (DIN), D16.2 (DOUT), D16.4 (DIN), D17.2 (DOUT), D17.4 (DIN), D19.2 (DOUT), D19.4 (DIN), D2.4 (DIN), D20.2 (DOUT), D20.4 (DIN), D22.2 (DOUT), D23.2 (DOUT), D7.2 (DOUT), D8.2 (DOUT)
- new net: D18.2 (DOUT), D21.4 (DIN)
- new net: D15.2 (DOUT), D18.4 (DIN)
- new net: D26.2 (DOUT), D27.4 (DIN)
- new net: D25.2 (DOUT), D26.4 (DIN)
- new net: D11.4 (DIN), D8.2 (DOUT)
- new net: D17.2 (DOUT), D20.4 (DIN)
- new net: D2.4 (DIN), D22.2 (DOUT)
- new net: D27.2 (DOUT), D28.4 (DIN)
- new net: D23.2 (DOUT), D3.4 (DIN)
- new net: D14.2 (DOUT), D17.4 (DIN)
- new net: D11.2 (DOUT), D14.4 (DIN)
- new net: D13.2 (DOUT), D16.4 (DIN)
- new net: D10.2 (DOUT), D13.4 (DIN)
- new net: D16.2 (DOUT), D19.4 (DIN)
- new net: D21.2 (DOUT), D24.4 (DIN)
- new net: D12.2 (DOUT), D15.4 (DIN)
- new net: D10.4 (DIN), D7.2 (DOUT)
- new net: D12.4 (DIN), D9.2 (DOUT)
- new net: D6.2 (DOUT), D9.4 (DIN)
- new net: D24.2 (DOUT), D25.4 (DIN)
- new net: D3.2 (DOUT), D6.4 (DIN)
- new net ADDRESSABLE_LED: U2.2 (1A)
- no-connect marks 0 -> 7
Other:
- company: Alex Goldberg -> Alex G
- title: MiniMixer -> @opensourcedj on twitter
- moved on the sheet: C10, C11, C13, C14, C16, C17, C19, C20, C22, C23, C25, C26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
